Commit message: Added gazebo world, gazebo control xacro file and launch file for all together

File: src/robot_description/description/robot.urdf.xacro (robot description, xacro)
@@ -2,3 +2,4 @@
 <robot xmlns:xacro="http://www.ros.org/wiki/xacro" name="robot">
     <xacro:include filename="robot_core.xacro"  />
+    <xacro:include filename="gazebo_control.xacro"  />
 </robot>

File: src/robot_description/description/robot_core.xacro (robot description, xacro)
@@ -41,4 +41,7 @@
         </xacro:inertial_cylinder>
     </link>
+    <gazebo reference="chassis">
+        <material>Gazebo/Black</material>
+    </gazebo>
     <!-- LEFT WHEEL LINK -->
     <joint name="left_wheel_joint" type="continuous">
@@ -64,4 +67,7 @@
         </xacro:inertial_cylinder>
     </link>
+    <gazebo reference="left_wheel">
+        <material>Gazebo/White</material>
+    </gazebo>
     <!-- RIGHT WHEEL LINK -->
     <joint name="right_wheel_joint" type="continuous">
@@ -87,4 +93,7 @@
         </xacro:inertial_cylinder>
     </link>
+    <gazebo reference="right_wheel">
+        <material>Gazebo/White</material>
+    </gazebo>
     <!-- CASTER WHEEL LINK -->
     <joint name="caster_wheel_joint" type="fixed">
@@ -109,3 +118,8 @@
         </xacro:inertial_sphere>
     </link>
+    <gazebo reference="caster_wheel">
+        <material>Gazebo/Red</material>
+        <mu1 value="0.001"/>
+        <mu2 value="0.001"/>
+    </gazebo>
 </robot>

Commit message: Added LiDAR to the sim model

File: src/robot_description/description/robot.urdf.xacro (robot description, xacro)
@@ -3,3 +3,4 @@
     <xacro:include filename="robot_core.xacro"  />
     <xacro:include filename="gazebo_control.xacro"  />
+    <xacro:include filename="lidar.xacro"/>
 </robot>

File: src/robot_description/description/robot_core.xacro (robot description, xacro)
@@ -48,5 +48,5 @@
         <parent link="base_link"/>
         <child link="left_wheel"/>
-        <origin rpy="-${pi/2} 0 0" xyz="0 0.12 0"/>
+        <origin rpy="-${pi/2} 0 0" xyz="0 0.12 0.0336"/>
         <axis xyz="0 0 1"/>
     </joint>
@@ -74,5 +74,5 @@
     <parent link="base_link"/>
         <child link="right_wheel"/>
-        <origin rpy="${pi/2} 0 0" xyz="0 -0.12 0"/>
+        <origin rpy="${pi/2} 0 0" xyz="0 -0.12 0.0336"/>
         <axis xyz="0 0 -1"/>
     </joint>
@@ -105,5 +105,5 @@
         <visual>
             <geometry>
-                <sphere radius="0.04"/>
+                <sphere radius="0.0114"/>
             </geometry>
             <material name="red"/>
@@ -111,8 +111,8 @@
         <collision>
             <geometry>
-                <sphere radius="0.04"/>
+                <sphere radius="0.0114"/>
             </geometry>
         </collision>
-        <xacro:inertial_sphere mass="0.1" radius="0.04">
+        <xacro:inertial_sphere mass="0.1" radius="0.0114">
             <origin rpy="0 0 0" xyz="0 0 0"/>
         </xacro:inertial_sphere>
