Commit message: Tested simulation, and deactivated plugings as any of them are working at the moment with gazebo

File: src/robot_description/description/lidar.xacro (robot description, xacro)
@@ -1,4 +1,4 @@
 <?xml version="1.0"?>
-<robot xmlns:xacro="http://www.ros.org/wiki/xacro" name="robot">
+<robot xmlns:xacro="http://www.ros.org/wiki/xacro">
     <joint name="laser_joint" type="fixed">
         <parent link="chassis"/>
@@ -41,5 +41,5 @@
                 </range>
             </ray>
-            <plugin name="laser_controller" filename="libgazebo_ros_laser.so">
+            <!-- <plugin name="laser_controller" filename="libgazebo_ros_laser.so">
                 <ros>
                   <namespace>/</namespace>
@@ -47,5 +47,5 @@
                 <topicName>scan</topicName>
                 <frameName>laser_frame</frameName>
-            </plugin>
+            </plugin> -->
         </sensor>
     </gazebo>

File: src/robot_description/description/robot.urdf.xacro (robot description, xacro)
@@ -1,7 +1,7 @@
 <?xml version="1.0"?>
 <robot xmlns:xacro="http://www.ros.org/wiki/xacro" name="robot">
-    <xacro:include filename="robot_core.xacro"  />
+    <xacro:include filename="robot_core.xacro"/>
+    <!-- <xacro:include filename="gazebo_control.xacro"  /> -->
     <xacro:include filename="ros2_control.xacro" />
-    <!-- <xacro:include filename="gazebo_control.xacro"  /> -->
     <xacro:include filename="lidar.xacro"/>
 </robot>

File: src/robot_description/description/robot_core.xacro (robot description, xacro)
@@ -1,4 +1,4 @@
-<?xml version="1.0" encoding="UTF-8"?>
-<robot xmlns:xacro="http://www.ros.org/wiki/xacro" name="robot">
+<?xml version="1.0"?>
+<robot xmlns:xacro="http://www.ros.org/wiki/xacro">
     <xacro:include filename="inertial_macros.xacro"/>
     <material name="black">
@@ -53,13 +53,13 @@
     <link name="left_wheel">
         <visual>
-          <geometry>
-            <cylinder length="0.015" radius="0.045"/>
-          </geometry>
-          <material name="white"/>
+            <geometry>
+                <cylinder length="0.015" radius="0.045"/>
+            </geometry>
+            <material name="white"/>
         </visual>
         <collision>
-          <geometry>
-            <cylinder length="0.015" radius="0.045"/>
-          </geometry>
+            <geometry>
+                <cylinder length="0.015" radius="0.045"/>
+            </geometry>
         </collision>
         <xacro:inertial_cylinder mass="0.1" length="0.015" radius="0.045">
@@ -72,5 +72,5 @@
     <!-- RIGHT WHEEL LINK -->
     <joint name="right_wheel_joint" type="continuous">
-    <parent link="base_link"/>
+        <parent link="base_link"/>
         <child link="right_wheel"/>
         <origin rpy="${pi/2} 0 0" xyz="0 -0.12 0.0336"/>
@@ -80,5 +80,5 @@
         <visual>
             <geometry>
-            <cylinder length="0.015" radius="0.045"/>
+                <cylinder length="0.015" radius="0.045"/>
             </geometry>
             <material name="white"/>
@@ -86,5 +86,5 @@
         <collision>
             <geometry>
-            <cylinder length="0.015" radius="0.045"/>
+                <cylinder length="0.015" radius="0.045"/>
             </geometry>
         </collision>

File: src/robot_description/description/ros2_control.xacro (robot description, xacro)
@@ -5,5 +5,5 @@
             <plugin>gazebo_ros2_control/GazeboSystem</plugin>
         </hardware>
-        <joint name ="left_wheel_joint">
+        <joint name="left_wheel_joint">
             <command_interface name="velocity">
                 <param name="min">-10</param>
@@ -13,5 +13,5 @@
             <state_interface name="position"/>
         </joint>
-        <joint name ="right_wheel_joint">
+        <joint name="right_wheel_joint">
             <command_interface name="velocity">
                 <param name="min">-10</param>
@@ -22,8 +22,10 @@
         </joint>
     </ros2_control>
-    <gazebo>
+    <!-- This plugin does not work for now, is crashing the sim and not
+     rendering anything -->
+    <!-- <gazebo>
         <plugin name="gazebo_ros2_control" filename="libgazebo_ros2_control.so">
             <parameters>$(find robot_description)/config/my_controllers.yaml</parameters>
         </plugin>
-    </gazebo>
+    </gazebo> -->
 </robot>

Commit message: Update the code to work with Humble

File: src/robot_description/description/lidar.xacro (robot description, xacro)
@@ -12,13 +12,13 @@
             </geometry>
             <material name="green"/>
-          </visual>
-          <collision>
+        </visual>
+        <collision>
             <geometry>
-              <cylinder length="0.056" radius="0.05"/>
+                <cylinder length="0.056" radius="0.05"/>
             </geometry>
-          </collision>
-          <xacro:inertial_cylinder mass="0.1" length="0.056" radius="0.05">
-              <origin rpy="0 0 0" xyz="0 0 0"/>
-          </xacro:inertial_cylinder>
+        </collision>
+        <xacro:inertial_cylinder mass="0.1" length="0.056" radius="0.05">
+            <origin rpy="0 0 0" xyz="0 0 0"/>
+        </xacro:inertial_cylinder>
     </link>
     <gazebo reference="laser_frame">
@@ -41,11 +41,11 @@
                 </range>
             </ray>
-            <!-- <plugin name="laser_controller" filename="libgazebo_ros_laser.so">
+            <plugin name="laser_controller" filename="libgazebo_ros_ray_sensor.so">
                 <ros>
-                  <namespace>/</namespace>
+                    <argument>~/out:=scan</argument>
                 </ros>
-                <topicName>scan</topicName>
-                <frameName>laser_frame</frameName>
-            </plugin> -->
+                <output_type>sensor_msgs/LaserScan</output_type>
+                <frame_name>laser_frame</frame_name>
+            </plugin>
         </sensor>
     </gazebo>

File: src/robot_description/description/robot.urdf.xacro (robot description, xacro)
@@ -1,7 +1,13 @@
 <?xml version="1.0"?>
 <robot xmlns:xacro="http://www.ros.org/wiki/xacro" name="robot">
+    <xacro:arg name="use_ros2_control" default="true"/>
+    <xacro:arg name="sim_mode" default="false"/>
     <xacro:include filename="robot_core.xacro"/>
-    <!-- <xacro:include filename="gazebo_control.xacro"  /> -->
-    <xacro:include filename="ros2_control.xacro" />
+    <xacro:if value="$(arg use_ros2_control)">
+        <xacro:include filename="ros2_control.xacro" />
+    </xacro:if>
+    <xacro:unless value="$(arg use_ros2_control)">
+        <xacro:include filename="gazebo_control.xacro" />
+    </xacro:unless>
     <xacro:include filename="lidar.xacro"/>
 </robot>

File: src/robot_description/description/ros2_control.xacro (robot description, xacro)
@@ -1,31 +1,64 @@
 <?xml version="1.0"?>
 <robot xmlns:xacro="http://www.ros.org/wiki/xacro">
-    <ros2_control name="GazeboSystem" type="system">
-        <hardware>
-            <plugin>gazebo_ros2_control/GazeboSystem</plugin>
-        </hardware>
-        <joint name="left_wheel_joint">
-            <command_interface name="velocity">
-                <param name="min">-10</param>
-                <param name="max">10</param>
-            </command_interface>
-            <state_interface name="velocity"/>
-            <state_interface name="position"/>
-        </joint>
-        <joint name="right_wheel_joint">
-            <command_interface name="velocity">
-                <param name="min">-10</param>
-                <param name="max">10</param>
-            </command_interface>
-            <state_interface name="velocity"/>
-            <state_interface name="position"/>
-        </joint>
-    </ros2_control>
+    <xacro:unless value="$(arg sim_mode)">
+        <ros2_control name="RealRobot" type="system">
+            <hardware>
+                <plugin>diffdrive_arduino/DiffDriveArduino</plugin>
+                <param name="left_wheel_name">left_wheel_joint</param>
+                <param name="right_wheel_name">right_wheel_joint</param>
+                <param name="loop_rate">30</param>
+                <param name="device">/dev/ttyACM0</param>
+                <param name="baud_rate">57600</param>
+                <param name="timeout">1000</param>
+                <param name="enc_counts_per_rev">1715</param>
+            </hardware>
+            <joint name="left_wheel_joint">
+                <command_interface name="velocity">
+                    <param name="min">-10</param>
+                    <param name="max">10</param>
+                </command_interface>
+                <state_interface name="velocity"/>
+                <state_interface name="position"/>
+            </joint>
+            <joint name="right_wheel_joint">
+                <command_interface name="velocity">
+                    <param name="min">-10</param>
+                    <param name="max">10</param>
+                </command_interface>
+                <state_interface name="velocity"/>
+                <state_interface name="position"/>
+            </joint>
+        </ros2_control>
+    </xacro:unless>
+    <xacro:if value="$(arg sim_mode)">
+        <ros2_control name="GazeboSystem" type="system">
+            <hardware>
+                <plugin>gazebo_ros2_control/GazeboSystem</plugin>
+            </hardware>
+            <joint name="left_wheel_joint">
+                <command_interface name="velocity">
+                    <param name="min">-10</param>
+                    <param name="max">10</param>
+                </command_interface>
+                <state_interface name="velocity"/>
+                <state_interface name="position"/>
+            </joint>
+            <joint name="right_wheel_joint">
+                <command_interface name="velocity">
+                    <param name="min">-10</param>
+                    <param name="max">10</param>
+                </command_interface>
+                <state_interface name="velocity"/>
+                <state_interface name="position"/>
+            </joint>
+        </ros2_control>
+    </xacro:if>
     <!-- This plugin does not work for now, is crashing the sim and not
      rendering anything -->
-    <!-- <gazebo>
+    <gazebo>
         <plugin name="gazebo_ros2_control" filename="libgazebo_ros2_control.so">
             <parameters>$(find robot_description)/config/my_controllers.yaml</parameters>
+            <parameters>$(find robot_description)/config/gaz_ros2_ctl_use_sim.yaml</parameters>
         </plugin>
-    </gazebo> -->
+    </gazebo>
 </robot>

Commit message: changed lidar yaw

File: src/robot_description/description/lidar.xacro (robot description, xacro)
@@ -4,5 +4,5 @@
         <parent link="chassis"/>
         <child link="laser_frame"/>
-        <origin rpy="0 0 0" xyz="-0.112 0.02 0.108"/>
+        <origin rpy="0 0 -${pi/2}" xyz="-0.112 0.02 0.108"/>
     </joint>
     <link name="laser_frame">

Commit message: Updated URDF description and controller config file to reflect more precise distances

File: src/robot_description/description/lidar.xacro (robot description, xacro)
@@ -4,5 +4,5 @@
         <parent link="chassis"/>
         <child link="laser_frame"/>
-        <origin rpy="0 0 -${pi/2}" xyz="-0.112 0.02 0.108"/>
+        <origin rpy="0 0 -1.4052" xyz="-0.112 0.02 0.108"/>
     </joint>
     <link name="laser_frame">

File: src/robot_description/description/robot_core.xacro (robot description, xacro)
@@ -54,5 +54,5 @@
         <visual>
             <geometry>
-                <cylinder length="0.015" radius="0.045"/>
+                <cylinder length="0.0147" radius="0.035"/>
             </geometry>
             <material name="white"/>
@@ -60,8 +60,8 @@
         <collision>
             <geometry>
-                <cylinder length="0.015" radius="0.045"/>
+                <cylinder length="0.0147" radius="0.035"/>
             </geometry>
         </collision>
-        <xacro:inertial_cylinder mass="0.1" length="0.015" radius="0.045">
+        <xacro:inertial_cylinder mass="0.1" length="0.147" radius="0.035">
             <origin rpy="0 0 0" xyz="0 0 0"/>
         </xacro:inertial_cylinder>
@@ -80,5 +80,5 @@
         <visual>
             <geometry>
-                <cylinder length="0.015" radius="0.045"/>
+                <cylinder length="0.0147" radius="0.035"/>
             </geometry>
             <material name="white"/>
@@ -86,8 +86,8 @@
         <collision>
             <geometry>
-                <cylinder length="0.015" radius="0.045"/>
+                <cylinder length="0.0147" radius="0.035"/>
             </geometry>
         </collision>
-        <xacro:inertial_cylinder mass="0.1" length="0.015" radius="0.045">
+        <xacro:inertial_cylinder mass="0.1" length="0.0147" radius="0.035">
             <origin rpy="0 0 0" xyz="0 0 0"/>
         </xacro:inertial_cylinder>

File: src/robot_description/description/ros2_control.xacro (robot description, xacro)
@@ -11,5 +11,5 @@
                 <param name="baud_rate">57600</param>
                 <param name="timeout">1000</param>
-                <param name="enc_counts_per_rev">1715</param>
+                <param name="enc_counts_per_rev">1716</param>
             </hardware>
             <joint name="left_wheel_joint">
