Commit message: Added an extra caster wheel to avoid unbalance when navigating

File: src/robot_description/description/robot_core.xacro (robot description, xacro)
@@ -96,5 +96,5 @@
         <material>Gazebo/White</material>
     </gazebo>
-    <!-- CASTER WHEEL LINK -->
+    <!-- FRONT CASTER WHEEL LINK -->
     <joint name="caster_wheel_joint" type="fixed">
         <parent link="chassis"/>
@@ -123,3 +123,30 @@
         <mu2 value="0.001"/>
     </gazebo>
+    <!-- BACK CASTER WHEEL LINK (Real robot does not have this, only for simulation purposes) -->
+    <joint name="back_caster_wheel_joint" type="fixed">
+        <parent link="chassis"/>
+        <child link="back_caster_wheel"/>
+        <origin xyz="-0.14 0 0"/>
+    </joint>
+    <link name="back_caster_wheel">
+        <visual>
+            <geometry>
+                <sphere radius="0.0114"/>
+            </geometry>
+            <material name="red"/>
+        </visual>
+        <collision>
+            <geometry>
+                <sphere radius="0.0114"/>
+            </geometry>
+        </collision>
+        <xacro:inertial_sphere mass="0.1" radius="0.0114">
+            <origin rpy="0 0 0" xyz="0 0 0"/>
+        </xacro:inertial_sphere>
+    </link>
+    <gazebo reference="back_caster_wheel">
+        <material>Gazebo/Red</material>
+        <mu1 value="0.001"/>
+        <mu2 value="0.001"/>
+    </gazebo>
 </robot>

Commit message: modified encoder counts per rev

File: src/robot_description/description/robot_core.xacro (robot description, xacro)
@@ -27,5 +27,5 @@
           <origin rpy="0 0 0" xyz="0 0 0.043"/>
           <geometry>
-            <cylinder length="0.08" radius="0.185"/>
+            <cylinder length="0.08" radius="0.171"/>
           </geometry>
           <material name="black"/>
@@ -34,8 +34,8 @@
           <origin rpy="0 0 0" xyz="0 0 0.043"/>
           <geometry>
-            <cylinder length="0.08" radius="0.185"/>
+            <cylinder length="0.08" radius="0171"/>
           </geometry>
         </collision>
-        <xacro:inertial_cylinder mass="3.6" length="0.08" radius="0.185">
+        <xacro:inertial_cylinder mass="3.6" length="0.08" radius="0.171">
             <origin rpy="0 0 0" xyz="0 0 0.043"/>
         </xacro:inertial_cylinder>

Commit message: Added Slam_toolbox config file, base_link, and a parameter wheel_radius to robot_core.xacro

File: src/robot_description/description/robot_core.xacro (robot description, xacro)
@@ -14,7 +14,14 @@
         <color rgba="0 1 0 1"/>
     </material>
+    <xacro:property name="wheel_radius" value="0.035"/>
     <!-- BASE LINK -->
     <link name="base_link">
     </link>
+    <!-- BASE_FOOTPRINT LINK -->
+    <joint name="base_footprint_joint" type="fixed">
+        <parent link="base_link"/>
+        <child link="base_footprint"/>
+        <origin rpy="0 0 0" xyz="0 0 0"/>
+    </joint>
     <!-- CHASSIS LINK -->
     <joint name="chassis_joint" type="fixed">
@@ -48,5 +55,5 @@
         <parent link="base_link"/>
         <child link="left_wheel"/>
-        <origin rpy="-${pi/2} 0 0" xyz="0 0.12 0.0336"/>
+        <origin rpy="-${pi/2} 0 0" xyz="0 0.12 ${wheel_radius - 0.0114}"/>
         <axis xyz="0 0 1"/>
     </joint>
@@ -54,5 +61,5 @@
         <visual>
             <geometry>
-                <cylinder length="0.0147" radius="0.035"/>
+                <cylinder length="0.0147" radius="${wheel_radius}"/>
             </geometry>
             <material name="white"/>
@@ -60,8 +67,8 @@
         <collision>
             <geometry>
-                <cylinder length="0.0147" radius="0.035"/>
+                <cylinder length="0.0147" radius="${wheel_radius}"/>
             </geometry>
         </collision>
-        <xacro:inertial_cylinder mass="0.1" length="0.147" radius="0.035">
+        <xacro:inertial_cylinder mass="0.1" length="0.147" radius="${wheel_radius}">
             <origin rpy="0 0 0" xyz="0 0 0"/>
         </xacro:inertial_cylinder>
@@ -74,5 +81,5 @@
         <parent link="base_link"/>
         <child link="right_wheel"/>
-        <origin rpy="${pi/2} 0 0" xyz="0 -0.12 0.0336"/>
+        <origin rpy="${pi/2} 0 0" xyz="0 -0.12 ${wheel_radius - 0.0114}"/>
         <axis xyz="0 0 -1"/>
     </joint>
@@ -80,5 +87,5 @@
         <visual>
             <geometry>
-                <cylinder length="0.0147" radius="0.035"/>
+                <cylinder length="0.0147" radius="${wheel_radius}"/>
             </geometry>
             <material name="white"/>
@@ -86,8 +93,8 @@
         <collision>
             <geometry>
-                <cylinder length="0.0147" radius="0.035"/>
+                <cylinder length="0.0147" radius="${wheel_radius}"/>
             </geometry>
         </collision>
-        <xacro:inertial_cylinder mass="0.1" length="0.0147" radius="0.035">
+        <xacro:inertial_cylinder mass="0.1" length="0.0147" radius="${wheel_radius}">
             <origin rpy="0 0 0" xyz="0 0 0"/>
         </xacro:inertial_cylinder>

Commit message: Implemented slam_toolbox and AMCL with Nav2

File: src/robot_description/description/robot_core.xacro (robot description, xacro)
@@ -24,4 +24,6 @@
         <origin rpy="0 0 0" xyz="0 0 0"/>
     </joint>
+    <link name="base_footprint">
+    </link>
     <!-- CHASSIS LINK -->
     <joint name="chassis_joint" type="fixed">
@@ -41,5 +43,5 @@
           <origin rpy="0 0 0" xyz="0 0 0.043"/>
           <geometry>
-            <cylinder length="0.08" radius="0171"/>
+            <cylinder length="0.08" radius="0.171"/>
           </geometry>
         </collision>
@@ -70,5 +72,5 @@
             </geometry>
         </collision>
-        <xacro:inertial_cylinder mass="0.1" length="0.147" radius="${wheel_radius}">
+        <xacro:inertial_cylinder mass="0.1" length="0.0147" radius="${wheel_radius}">
             <origin rpy="0 0 0" xyz="0 0 0"/>
         </xacro:inertial_cylinder>
